Commit message: Update

File: yolo_landmark/urdf/test_diff_drive.xacro.urdf (robot description, URDF)
Before this commit: robot diff_drive, 5 links, 4 joints
Links:
- removed link chassis
- added link base_link, mass 1.14395; collision box size=2.01142 1 0.568726; visual box size=2.01142 1 0.568726
- added link lidar_link, mass 0.1; collision cylinder length=0.3 radius=0.2; visual cylinder length=0.3 radius=0.2
- link camera_link: geometry collision box size=0.3 0.3 0.2; visual box size=0.3 0.3 0.2
Joints:
- added joint lidar_joint: type fixed, parent base_link, child lidar_link, origin xyz=0.0 0 0.9 rpy=0 0 0
- joint camera_joint: origin xyz=1.0 0 0.8 rpy=0 0 0 -> xyz=1.0 0 0.55 rpy=0 0 0; parent chassis -> base_link
- joint caster_joint: parent chassis -> base_link
- joint left_wheel_joint: parent chassis -> base_link
- joint right_wheel_joint: parent chassis -> base_link

Commit message: Update

File: yolo_landmark/urdf/test_diff_drive.xacro.urdf (robot description, URDF)
Before this commit: robot diff_drive, 6 links, 5 joints
Links:
- link caster: mass 0.005 -> 0.2

Commit message: mapping

File: yolo_landmark/urdf/test_diff_drive.xacro.urdf (robot description, URDF)
Before this commit: robot diff_drive, 6 links, 5 joints
Links:
- link base_link: mass 1.14395 -> 3; geometry collision box size=0.8 0.4 0.2; visual box size=0.8 0.4 0.2
- link camera_link: mass 0.1 -> 0.3; geometry collision box size=0.2 0.2 0.2; visual box size=0.2 0.2 0.2
- link caster: mass 0.2 -> 0.5; geometry collision sphere radius=0.1; visual sphere radius=0.1
- link left_wheel: mass 2 -> 0.3; geometry collision cylinder length=0.1 radius=0.1; visual cylinder length=0.1 radius=0.1
- link lidar_link: mass 0.1 -> 0.2; geometry collision cylinder length=0.1 radius=0.1; visual cylinder length=0.1 radius=0.1
- link right_wheel: mass 2 -> 0.5; geometry collision cylinder length=0.1 radius=0.1; visual cylinder length=0.1 radius=0.1
Joints:
- joint camera_joint: origin xyz=1.0 0 0.55 rpy=0 0 0 -> xyz=0.41 0 0 rpy=0 0 0
- joint caster_joint: origin xyz=-0.957138 -0 0.2 rpy=0 0 0 -> xyz=-0.3 0 -0.1 rpy=0 0 0
- joint left_wheel_joint: origin xyz=0.554283 0.625029 0.3 rpy=-1.5707 0 0 -> xyz=0.2 0.25 -0.1 rpy=-1.5707 0 0
- joint lidar_joint: origin xyz=0.0 0 0.9 rpy=0 0 0 -> xyz=0.0 0 0.15 rpy=0 0 0
- joint right_wheel_joint: origin xyz=0.554283 -0.625029 0.3 rpy=-1.5707 0 0 -> xyz=0.2 -0.25 -0.1 rpy=-1.5707 0 0

Commit message: Fixed sdf and urdf

File: yolo_landmark/urdf/test_diff_drive.xacro.urdf (robot description, URDF)
Before this commit: robot diff_drive, 6 links, 5 joints
Links:
- link base_link: mass 3 -> 1.14395; geometry collision box size=2.01142 1 0.568726; visual box size=2.01142 1 0.568726
- link camera_link: mass 0.3 -> 0.01
- link caster: mass 0.5 -> 0.005; geometry collision sphere radius=0.2; visual sphere radius=0.2
- link left_wheel: mass 0.3 -> 2; geometry collision sphere radius=0.3; visual sphere radius=0.3
- link lidar_link: mass 0.2 -> 0.01
- link right_wheel: mass 0.5 -> 2; geometry collision sphere radius=0.3; visual sphere radius=0.3
Joints:
- joint camera_joint: origin xyz=0.41 0 0 rpy=0 0 0 -> xyz=0.848573 0 0.65 rpy=0 0 0
- joint caster_joint: origin xyz=-0.3 0 -0.1 rpy=0 0 0 -> xyz=-0.957138 0 0.2 rpy=0 0 0
- joint left_wheel_joint: origin xyz=0.2 0.25 -0.1 rpy=-1.5707 0 0 -> xyz=0.554283 0.625029 0.3 rpy=-1.5707 0 0
- joint lidar_joint: origin xyz=0.0 0 0.15 rpy=0 0 0 -> xyz=0.648573 0 0.81 rpy=0 0 0
- joint right_wheel_joint: origin xyz=0.2 -0.25 -0.1 rpy=-1.5707 0 0 -> xyz=0.554283 -0.625029 0.3 rpy=-1.5707 0 0

Commit message: Update

File: yolo_landmark/urdf/test_diff_drive.xacro.urdf (robot description, URDF)
Before this commit: robot diff_drive, 6 links, 5 joints
Joints:
- joint camera_joint: origin xyz=0.848573 0 0.65 rpy=0 0 0 -> xyz=0.8 0 0.15 rpy=0 0 0
- joint caster_joint: origin xyz=-0.957138 0 0.2 rpy=0 0 0 -> xyz=-0.805711 0 -0.3 rpy=0 0 0
- joint left_wheel_joint: origin xyz=0.554283 0.625029 0.3 rpy=-1.5707 0 0 -> xyz=0.70571 0.625029 -0.2 rpy=-1.5707 0 0
- joint lidar_joint: origin xyz=0.648573 0 0.81 rpy=0 0 0 -> xyz=0.8 0 0.31 rpy=0 0 0
- joint right_wheel_joint: origin xyz=0.554283 -0.625029 0.3 rpy=-1.5707 0 0 -> xyz=0.70571 -0.625029 -0.2 rpy=-1.5707 0 0
